Commit message: Final Code Before Testing Terkiz

File: install/kal_package/share/kal_package/src/description/ros2_control.xacro (robot description, xacro)
@@ -8,5 +8,5 @@
       <param name="right_wheel_name">drivewhl_r_joint</param>
       <param name="loop_rate">30</param>
-      <param name="device">/dev/ttyACM0</param>
+      <param name="device">/dev/serial/by-id/usb-Arduino__www.arduino.cc__0042_95735343633351C021B2-if00</param>
       <param name="baud_rate">57600</param>
       <param name="timeout_ms">1000</param>

File: install/kal_package/share/kal_package/src/description/wheels.xacro (robot description, xacro)
@@ -46,5 +46,5 @@
     <parent link="base_link"/>
     <child link="caster_wheel"/>
-    <origin xyz="-0.06 0 -0.0225"/>
+    <origin xyz="0.06 0 -0.0225"/>
   </joint>
   <link name="caster_wheel">
